File: NAND_flash_chip_sketch.kicad_sch (KiCad schematic)
At the start: 1 part, among them U7 AS5F31G04SND-08LIN

Commit message: Corrected footprint assignment errors
Parts:
- U7: footprint AS5F31G04SND-08LIN:SON127P600X800X80-8N -> footprints:SON127P600X800X80-8N
Changed lines of the file:
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@@
 			)
 		)
-		(property "Footprint" "AS5F31G04SND-08LIN:SON127P600X800X80-8N"
+		(property "Footprint" "footprints:SON127P600X800X80-8N"
 			(at 127 83.82 0)
 			(effects
