File: accelerometer_sketch.kicad_sch (KiCad schematic)
At the start: 3 parts, among them U6 KX134-1211

Commit message: Corrected footprint assignment errors
Parts:
- U6: footprint LGA12_2X2X0P9_ROM -> footprints:LGA12_2X2X0P9_ROM
Changed lines of the file:
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@@
 			)
 		)
-		(property "Footprint" "LGA12_2X2X0P9_ROM"
+		(property "Footprint" "footprints:LGA12_2X2X0P9_ROM"
 			(at 105.41 66.04 0)
 			(effects
