File: gyroscope_sketch.kicad_sch (KiCad schematic)
At the start: 3 parts, among them U5 ASM330LHH

Commit message: Corrected footprint assignment errors
Parts:
- U5: footprint LGA-14L_2P5X3X0P83_STM -> footprints:LGA-14L_2P5X3X0P83_STM
Changed lines of the file:
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@@
 			)
 		)
-		(property "Footprint" "LGA-14L_2P5X3X0P83_STM"
+		(property "Footprint" "footprints:LGA-14L_2P5X3X0P83_STM"
 			(at 106.68 68.58 0)
 			(effects
