File: magnometer_sketch.kicad_sch (KiCad schematic)
At the start: 2 parts, among them U4 MMC5983MA

Commit message: Corrected footprint assignment errors
Parts:
- U4: footprint MMC5983MA_MEM -> footprints:MMC5983MA_MEM
Changed lines of the file:
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@@
 			)
 		)
-		(property "Footprint" "MMC5983MA_MEM"
+		(property "Footprint" "footprints:MMC5983MA_MEM"
 			(at 81.28 64.77 0)
 			(effects
