File: SRAD_V2/SRAD_V2.kicad_sch (KiCad schematic)
At the start: 44 parts, among them SW1 SW_Push_Dual, SW2 SW_Nidec_CAS-120A1, U1 STM32F767ZIT6, U11 KX134-1211, U12 MAX-M10S, U13 MS5607-02BA, U14 MMC5983MA, U15 ASM330LHH, U16 MCP9808_DFN, U17 AS5F31G04SND-08LIN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

Commit message: Sensor routing and integration of various systems on the PCB
Connections:
- net IMU_SPI_SDO: no longer U1.112 (PC11)
- net MAG_SPI_SDO: now also U1.112 (PC11)
Changed lines of the file:
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@@
 		)
 	)
-	(global_label "IMU_SPI_SDO"
+	(global_label "MAG_SPI_SDO"
 		(shape input)
 		(at 118.11 205.74 0)
@@
 		)
 		(property "Intersheetrefs" "${INTERSHEET_REFS}"
-			(at 133.3114 205.74 0)
+			(at 133.7347 205.74 0)
 			(hide yes)
 			(show_name no)

Commit message: more routing
Parts:
- added C40, C41: C_Polarized, symbol Device:C_Polarized
Connections:
- net GND: now also C40.2, C41.2
- new net +BATT: C40.1, C41.1
Other:
- sheet E-match Firing Circuit ports: added +BATT; removed VBAT
- sheet Power Delivery System ports: added +3.3V; removed +3V3
- moved on the sheet: BZ1

Commit message: Updated the buzzer
Parts:
- removed BZ1: Buzzer, buzzer:XDCR_AI-3035-TWT-3V-R, symbol Device:Buzzer
- removed C12, C13, C19: 100n, Capacitor_SMD:C_0603_1608Metric, symbol Device:C_Small
- removed C14: 10u, Capacitor_SMD:C_0603_1608Metric, symbol Device:C_Small
- removed U11: KX134-1211, footprints:LGA12_2X2X0P9_ROM, symbol KX134-1211:KX134-1211
- removed U15: ASM330LHH, footprints:LGA-14L_2P5X3X0P83_STM, symbol ASM330LHH:ASM330LHH
- removed U16: MCP9808_DFN, Package_DFN_QFN:DFN-8-1EP_3x2mm_P0.5mm_EP1.7x1.4mm, symbol Sensor_Temperature:MCP9808_DFN
- added BZ2: Buzzer, Buzzer_Beeper:MagneticBuzzer_StarMicronics_HMB-06_HMB-12, symbol Device:Buzzer
Connections:
- net GND: now also BZ2.2 (-)
Other:
- note added: "BUZZER"
- note added: "Bulk Capacitance"
- note removed: "ACCELEROMETER"
- note removed: "Gyro"
- note removed: "TEMPERATURE"
- moved on the sheet: C40, C41
