File: Breakout Boards/breakout_boards.kicad_sch (KiCad schematic)
At the start: 4 parts

Commit message: Updated the 3.3V test point
Parts:
- added D1, D3: 1N914, Diode_THT:D_DO-35_SOD27_P7.62mm_Horizontal, symbol Diode:1N914
Connections:
- new net V1: D1.2 (A)
- new net V2: D3.2 (A)
- new net Vout: D1.1 (K), D3.1 (K)
