File: Breakout Boards/breakout_boards.kicad_pcb (KiCad board)
At the start: 4 copper layers, 72.5 x 61.5 mm, 54 parts, among them J10 Conn_01x04_Pin, J11 Conn_01x04_Pin, J12 Conn_01x04_Pin, J13 Conn_01x04_Pin, J14 Conn_01x04_Pin, J15 Conn_01x04_Pin, J16 Conn_01x04_Pin, J17 Conn_01x04_Pin, J18 Conn_01x04_Pin, J19 Conn_01x04_Pin, J9 Conn_01x04_Pin, Q5 NPN BJT

Commit message: Updated the 3.3V test point
Other:
- board text removed: "V1.0"
Changed lines of the file:
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@@
-		)
-	)
-	(gr_text "V1.0"
-		(at 90.2 63.8 0)
-		(layer "F.SilkS")
-		(effects
-			(font
-				(size 1 1)
-				(thickness 0.2)
-				(bold yes)
-			)
-			(justify left bottom)
 		)
 	)

Commit message: Created a PCB layout for the Barometer
Parts:
- moved J12 80.2 mm to (115.5, 99.5)
- moved J13 76.8 mm to (93.5, 107.5), turned to 180 degrees
- moved J15 76.3 mm to (54.5, 81.0)
- moved J17 70.8 mm to (76.5, 88.5), turned to 180 degrees
- moved C33 3.46 mm to (108.5, 102.3), turned to -90 degrees
- moved kibuzzard-6A982418 2.89 mm to (67.7, 89.7)
- moved IC5 2.58 mm to (101.2, 103.0)
- moved kibuzzard-6A6394C9 2.00 mm to (101.5, 111.0)
- moved C31 1.63 mm to (111.0, 102.3), turned to 90 degrees
Connections:
- J12 pad 1: unconnected-(J12-Pin_1-Pad1) -> +3.3V
- J12 pad 3: unconnected-(J12-Pin_3-Pad3) -> NAND_SPI_IO3
- J12 pad 4: +3.3V -> NAND_SPI_IO2
- J13 pad 1: unconnected-(J13-Pin_1-Pad1) -> NAND_SPI_IO0
- J13 pad 2: GND -> NAND_SPI_CLK
- J13 pad 3: unconnected-(J13-Pin_3-Pad3) -> NAND_SPI_IO1
- J13 pad 4: +3.3V -> NAND_SPI_CS
- J15 pad 1: unconnected-(J15-Pin_1-Pad1) -> BAR_SPI_CS
- J15 pad 2: GND -> BAROMETER_MISO
- J15 pad 3: unconnected-(J15-Pin_3-Pad3) -> BAROMETER_MOSI
- J15 pad 4: +3.3V -> BAROMETER_SCLK
- J17 pad 2: GND -> unconnected-(J17-Pin_1-Pad1)
- J17 pad 3: unconnected-(J17-Pin_3-Pad3) -> GND
Routing:
- net GND: track 48.9 -> 85.7 mm
- net NAND_SPI_IO2: track 1.85 -> 21.9 mm, vias 0 -> 1
- net NAND_SPI_IO0: track 3.76 -> 15.0 mm, vias 0 -> 1
- net BAR_SPI_CS: track 3.10 -> 12.0 mm
- net BAROMETER_SCLK: track 5.57 -> 13.7 mm
- net +3.3V: track 88.9 -> 94.8 mm
- net BAROMETER_MOSI: track 7.12 -> 12.5 mm
- net NAND_SPI_CS: track 7.88 -> 4.38 mm, vias 1 -> 0
- net NAND_SPI_IO3: track 8.85 -> 11.3 mm
- net BAROMETER_MISO: track 9.61 -> 11.9 mm
- net NAND_SPI_CLK: track 12.0 -> 14.0 mm, vias 0 -> 1
- net NAND_SPI_IO1: track 2.81 -> 3.88 mm
Other:
- board text added: "MISO"
- board text added: "MOSI"
- board text added: "SCLK"
- board text added: "SPI"
